File: task_6_PDB/Power_Distro_PCB.brd (EAGLE design)
At the start: 101.6 x 63.6 mm, 52 parts

Commit message: layout and labels done
Parts:
- TVS_1, TVS_8: value 26V_TVS -> 26V
- TVS_2, TVS_5: value SMBJ3V3_TVSSMB -> 3V3
- TVS_3, TVS_6: value SMAJ5.0_TVSSMA -> 5V
- TVS_4, TVS_7: value PRSMA16_TVS -> 16V
- VREG_1: value 29300-3.3WU -> 3V3
- VREG_2: value 29300-5.0WU -> 5V
- VREG_3: value 29300-12WU -> 12V
- VREG_4, VREG_5, VREG_6: value MIC29300-3.3WU -> 3V3
- VREG_7: value MIC2900-3.3WU -> 3V3
- moved TVS_4 4.95 mm to (78.5, 5.84)
- moved F5 3.95 mm to (78.9, 10.9)
- moved TVS_2 3.05 mm to (78.7, 21.0)
- moved TVS_7 2.80 mm to (78.7, 16.1)
- moved F3 2.03 mm to (78.9, 26.5)
- moved TVS_6 1.55 mm to (78.9, 47.4)
- moved TVS_5 1.27 mm to (78.9, 32.1)
- moved TVS_3 0.68 mm to (78.9, 37.1)
- moved F4 0.46 mm to (78.9, 42.2)
- renumbered 12V_LO_IND to 12V, 3.3V_IND to 3.3V, 5V_IND to 5V, MOTOR_IND to MOTOR, PWR_IN_IND to PWR
Routing:
- net 24V_REG: track 200.0 -> 226.0 mm, vias 0 -> 2
- net N$1: track 21.4 -> 42.7 mm, vias 0 -> 2
- net N$3: track 19.2 -> 38.1 mm
- net GND: track 304.1 -> 310.5 mm
- net 24V_REG_MOTOR: track 93.6 -> 98.3 mm
- net N$10: track 17.4 -> 19.6 mm
- net N$6: track 17.5 -> 19.5 mm
- net 5V_REG: track 117.7 -> 116.1 mm
- net 3.3V_REG: track 94.0 -> 92.9 mm
- net N$7: track 17.5 -> 18.2 mm
- net N$4: track 6.68 -> 7.44 mm
- net N$11: track 6.41 -> 7.16 mm
- net 12V_REG: track 72.8 -> 72.0 mm
- net N$17: track 6.41 -> 7.16 mm
Other:
- board text added: "Team B : Aaron Basel David Edward Georgia"
