File: task_6_PDB/Power_Distro_PCB.sch (EAGLE design)
At the start: 52 parts

Commit message: layout and labels done
Parts:
- TVS_1, TVS_8: value 26V_TVS -> 26V
- TVS_2, TVS_5: value SMBJ3V3_TVSSMB -> 3V3
- TVS_3, TVS_6: value SMAJ5.0_TVSSMA -> 5V
- TVS_4, TVS_7: value PRSMA16_TVS -> 16V
- VREG_1: value 29300-3.3WU -> 3V3
- VREG_2: value 29300-5.0WU -> 5V
- VREG_3: value 29300-12WU -> 12V
- VREG_4, VREG_5, VREG_6: value MIC29300-3.3WU -> 3V3
- VREG_7: value MIC2900-3.3WU -> 3V3
- renumbered 12V_LO_IND to 12V, 3.3V_IND to 3.3V, 5V_IND to 5V, MOTOR_IND to MOTOR, PWR_IN_IND to PWR
