File: task_6_PDB/V2.0/Power_Distro_PCB.brd (EAGLE design)
At the start: 101.6 x 63.6 mm, 52 parts

Commit message: finished V2.0, corrected values and overall
Parts:
- removed 12V_LO_IND, 3.3V_IND, 5V_IND, MOTOR_IND: GREEN, led:SML1206
- removed C10, C12, C14: 10uF, resistor:C1206
- removed C11, C13, C16, C9: 33uF, resistor:C1206
- removed C15: 100uF, resistor:C1206
- removed PWR_IN_IND: RED, led:SML1206
- removed VREG_4, VREG_5, VREG_6: MIC29300-3.3WU, POWER_DISTRO:TO-263-3
- removed VREG_7: MIC2900-3.3WU, POWER_DISTRO:TO-263-3
- added 12V, 3.3V, 5V, MOTOR, POWER: GREEN, led:SML1206
- C1: value 33uF -> 150uF
- C2: value 10uF -> 100uF
- C3, C5, C6, C7: value 33uF -> 10uF
- F3: value 3.3V_1A -> 12V_2A
- F5: value 12V_2A -> 3.3V_1A
- R1, R2: value 47 -> 1100
- R3: value 47 -> 500
- R4: value 47 -> 150
- R5: value 47 -> 65
- TVS_1: value 26V_TVS -> 26V
- TVS_2: value SMBJ3V3_TVSSMB -> 26V; device POWER_DISTRO:DO-214AA -> POWER_DISTRO:DO-214AC
- TVS_3: value SMAJ5.0_TVSSMA -> 16V
- TVS_4: value PRSMA16_TVS -> 16V
- TVS_5: value SMBJ3V3_TVSSMB -> 5V; device POWER_DISTRO:DO-214AA -> POWER_DISTRO:DO-214AC
- TVS_6: value SMAJ5.0_TVSSMA -> 5V
- TVS_7: value PRSMA16_TVS -> 3V3; device POWER_DISTRO:DO-214AC -> POWER_DISTRO:DO-214AA
- TVS_8: value 26V_TVS -> 3V3; device POWER_DISTRO:DO-214AC -> POWER_DISTRO:DO-214AA
- VREG_1: value 29300-3.3WU -> 12V
- VREG_2: value 29300-5.0WU -> 5V
- VREG_3: value 29300-12WU -> 3V3
- moved TVS_2 60.4 mm to (26.8, 55.1), turned to 270 degrees
- moved TVS_3 49.7 mm to (40.6, 5.59), turned to 0 degrees
- moved C2 47.8 mm to (31.1, 54.9)
- moved C1 45.8 mm to (11.2, 55.0), turned to 90 degrees
- moved C4 45.6 mm to (34.7, 14.9), turned to 270 degrees
- moved C6 45.1 mm to (34.5, 41.3), turned to 270 degrees
- moved C5 44.9 mm to (17.1, 46.9), turned to 180 degrees
- moved F3 42.0 mm to (40.8, 10.9)
- moved F5 39.6 mm to (40.8, 26.5)
- moved TVS_5 38.4 mm to (40.6, 36.8), turned to 0 degrees
- moved C3 38.4 mm to (17.1, 20.1), turned to 180 degrees
- moved TVS_4 38.3 mm to (40.6, 16.1)
- moved CPU_OUT 38.1 mm to (55.2, 24.3)
- moved ENCODER_OUT 38.1 mm to (55.2, 42.8)
- moved LIDAR_OUT 38.1 mm to (55.2, 14.9)
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Connections:
- removed net 3.3V_REG: CPU_OUT.1, R1.2, TVS_5.1
- removed net N$12: PWR_IN_IND.A, R5.1
- removed net N$13: C8.2, R5.2, VREG_4.3
- removed net N$14: C10.2, R2.2, VREG_5.3
- removed net N$15: C12.2, R3.2, VREG_6.3
- removed net N$16: C14.2, R4.2, VREG_7.3
- new net N$18: 3.3V.A, R5.1
- new net N$20: 5V.A, R4.1
- net 12V_REG: now also R3.1, TVS_4.1; no longer C11.2, TVS_7.1, VREG_6.1
- net 24V_REG: now also C2.2, TVS_2.1; no longer C1.2, C16.2, TVS_8.1, VREG_4.1
- net 24V_REG_MOTOR: now also R2.1; no longer C13.2, VREG_7.1
- net 5V_REG: now also R4.2; no longer C9.2, VREG_5.1
- net GND: now also 12V.C, 3.3V.C, 5V.C, MOTOR.C, POWER.C, TVS_5.2, TVS_7.2; no longer 12V_LO_IND.C, 3.3V_IND.C, 5V_IND.C, C10.1, C11.1, C12.1, C13.1, C14.1, C15.1, C16.1, C9.1, MOTOR_IND.C, PWR_IN_IND.C, TVS_1.2, TVS_4.2, VREG_4.2, VREG_4.4, VREG_5.2, VREG_5.4, VREG_6.2, VREG_6.4, VREG_7.2, VREG_7.4
- net N$1: now also POWER.A, R1.2; no longer F1.2, TVS_8.2
- net N$10: now also C4.2, F3.1, TVS_3.1, VREG_1.3; no longer C6.2, F5.1, TVS_4.1, VREG_3.3
- net N$17: now also F3.2, TVS_4.2; no longer F5.2, TVS_7.2
- net N$2: now also 12V.A, R3.2; no longer 3.3V_IND.A, R1.1
- net N$3: now also C1.2; no longer C15.2
- net N$4: now also F5.2, TVS_8.2; no longer F3.2, TVS_5.2
- net N$5: now also CPU_OUT.1, R5.2, TVS_8.1; no longer 5V_IND.A, R2.1
- net N$6: now also C8.2, F5.1, TVS_7.1, VREG_3.3; no longer C2.2, F3.1, TVS_2.1, VREG_1.3
- net N$7: now also C6.2, TVS_5.1; no longer C4.2, TVS_3.1
- net N$8: now also MOTOR.A, R2.2; no longer 12V_LO_IND.A, R3.1
- net N$9: now also F1.2, R1.1, TVS_1.2; no longer MOTOR_IND.A, R4.1
Routing:
- net 24V_REG: track 200.0 -> 84.9 mm, vias 0 -> 2
- net 3.3V_REG: track 94.0 -> 0.00 mm, vias 1 -> 0
- net N$15: track 53.3 -> 0.00 mm
- net N$13: track 52.6 -> 0.00 mm
- net GND: track 266.6 -> 214.9 mm, vias 9 -> 29
- net N$5: track 6.77 -> 55.7 mm, vias 0 -> 1
- net 5V_REG: track 117.7 -> 74.7 mm
- net N$14: track 39.6 -> 0.00 mm
- net N$9: track 6.77 -> 44.8 mm, vias 0 -> 2
- net 24V_REG_MOTOR: track 93.6 -> 64.8 mm
- net N$16: track 26.3 -> 0.00 mm
- net N$1: track 21.4 -> 3.31 mm
- net N$10: track 17.4 -> 31.9 mm
- net N$7: track 17.5 -> 31.9 mm
- net N$6: track 17.5 -> 31.2 mm
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Other:
- board size 101.6 x 63.6 mm -> 63.5 x 63.6 mm
- board text added: "Team B : Aaron Basel David Edward Georgia"
