File: task_6_PDB/V2.0/Power_Distro_PCB.sch (EAGLE design)
At the start: 52 parts

Commit message: finished V2.0, corrected values and overall
Parts:
- removed 12V_LO_IND, 3.3V_IND, 5V_IND, MOTOR_IND: GREEN, led:LEDSML1206
- removed C10, C12, C14: 10uF, resistor:C-EUC1206
- removed C11, C13, C16, C9: 33uF, resistor:C-EUC1206
- removed C15: 100uF, resistor:C-EUC1206
- removed PWR_IN_IND: RED, led:LEDSML1206
- removed VREG_4, VREG_5, VREG_6: MIC29300-3.3WU, POWER_DISTRO:HIGH-CURRENT_REGSMA
- removed VREG_7: MIC2900-3.3WU, POWER_DISTRO:HIGH-CURRENT_REGSMA
- added 12V, 3.3V, 5V, MOTOR, POWER: GREEN, led:LEDSML1206
- C1: value 33uF -> 150uF
- C2: value 10uF -> 100uF
- C3, C5, C6, C7: value 33uF -> 10uF
- F3: value 3.3V_1A -> 12V_2A
- F5: value 12V_2A -> 3.3V_1A
- R1, R2: value 47 -> 1100
- R3: value 47 -> 500
- R4: value 47 -> 150
- R5: value 47 -> 65
- TVS_1: value 26V_TVS -> 26V
- TVS_2: value SMBJ3V3_TVSSMB -> 26V; device POWER_DISTRO:SMBJ3V3_TVSSMB -> POWER_DISTRO:SMAJ26A_TVSSMA
- TVS_3: value SMAJ5.0_TVSSMA -> 16V; device POWER_DISTRO:SMAJ5.0_TVSSMA -> POWER_DISTRO:PRSMA16_TVS
- TVS_4: value PRSMA16_TVS -> 16V
- TVS_5: value SMBJ3V3_TVSSMB -> 5V; device POWER_DISTRO:SMBJ3V3_TVSSMB -> POWER_DISTRO:SMAJ5.0_TVSSMA
- TVS_6: value SMAJ5.0_TVSSMA -> 5V
- TVS_7: value PRSMA16_TVS -> 3V3; device POWER_DISTRO:PRSMA16_TVS -> POWER_DISTRO:SMBJ3V3_TVSSMB
- TVS_8: value 26V_TVS -> 3V3; device POWER_DISTRO:SMAJ26A_TVSSMA -> POWER_DISTRO:SMBJ3V3_TVSSMB
- VREG_1: value 29300-3.3WU -> 12V
- VREG_2: value 29300-5.0WU -> 5V
- VREG_3: value 29300-12WU -> 3V3
Connections:
- removed net 3.3V_REG: CPU_OUT-1.S, R1.2, TVS_5.CATHODE
- removed net N$12: PWR_IN_IND.A, R5.1
- removed net N$13: C8.2, R5.2, VREG_4.OUT
- removed net N$14: C10.2, R2.2, VREG_5.OUT
- removed net N$15: C12.2, R3.2, VREG_6.OUT
- removed net N$16: C14.2, R4.2, VREG_7.OUT
- new net N$18: 3.3V.A, R5.1
- new net N$20: 5V.A, R4.1
- net 12V_REG: now also R3.1, TVS_4.CATHODE; no longer C11.2, TVS_7.CATHODE, VREG_6.IN
- net 24V_REG: now also C2.2, TVS_2.CATHODE; no longer C1.2, C16.2, TVS_8.CATHODE, VREG_4.IN
- net 24V_REG_MOTOR: now also R2.1; no longer C13.2, VREG_7.IN
- net 5V_REG: now also R4.2; no longer C9.2, VREG_5.IN
- net GND: now also 12V.C, 3.3V.C, 5V.C, MOTOR.C, POWER.C, TVS_5.ANODE, TVS_7.ANODE; no longer 12V_LO_IND.C, 3.3V_IND.C, 5V_IND.C, C10.1, C11.1, C12.1, C13.1, C14.1, C15.1, C16.1, C9.1, MOTOR_IND.C, PWR_IN_IND.C, TVS_1.ANODE, TVS_4.ANODE, VREG_4.GND, VREG_5.GND, VREG_6.GND, VREG_7.GND
- net N$1: now also POWER.A, R1.2; no longer F1.2, TVS_8.ANODE
- net N$10: now also C4.2, F3.1, TVS_3.CATHODE, VREG_1.OUT; no longer C6.2, F5.1, TVS_4.CATHODE, VREG_3.OUT
- net N$17: now also F3.2, TVS_4.ANODE; no longer F5.2, TVS_7.ANODE
- net N$2: now also 12V.A, R3.2; no longer 3.3V_IND.A, R1.1
- net N$3: now also C1.2; no longer C15.2
- net N$4: now also F5.2, TVS_8.ANODE; no longer F3.2, TVS_5.ANODE
- net N$5: now also CPU_OUT-1.S, R5.2, TVS_8.CATHODE; no longer 5V_IND.A, R2.1
- net N$6: now also C8.2, F5.1, TVS_7.CATHODE, VREG_3.OUT; no longer C2.2, F3.1, TVS_2.CATHODE, VREG_1.OUT
- net N$7: now also C6.2, TVS_5.CATHODE; no longer C4.2, TVS_3.CATHODE
- net N$8: now also MOTOR.A, R2.2; no longer 12V_LO_IND.A, R3.1
- net N$9: now also F1.2, R1.1, TVS_1.ANODE; no longer MOTOR_IND.A, R4.1
Other:
- note added: "LED specs are 2V forward voltage with 20mA recommended current."
- note removed: "Indicator LEDs"
- moved on the sheet: C1, C2, C3, C4, C5, C6, C7, C8, F3, F5, R1, R2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
