File: task_12_PDS PCB/Power_Distro_Board.brd (EAGLE design)
At the start: 63.5 x 63.6 mm, 35 parts

Commit message: PCB sch done, added another lib called minebot_PDR.lbr
Parts:
- removed 12V, 5V, STEPPER: GREEN, led:SML1206
- removed AUX, GPS_OUT: C-GRID-02-70543, con-molex:70543-02
- removed DCMOTOR_OUT, STEPPER_OUT: 5566-2, con-molex:5566-2
- removed R3: 500, resistor:R1206
- removed TVS_4: 16V, diode:SMC
- removed TVS_6: 5V, diode:SMC
- added 12V_3A, 12V_5A, STEPPER_OUT_1, STEPPER_OUT_2, STEPPER_OUT_3: 5566-2, con-molex:5566-2
- added 12V_3A_, 12V_5A_, OUT_5V, RAIL_5V, RPI_5V, STEPPER_1, STEPPER_2, STEPPER_3: GREEN, led:SML1206
- added 5V_OUT: C-GRID-02-70543, con-molex:70543-02
- added 5V_RAIL: 5v, pinhead:2X05
- added C1_1, C2_1, C3_1: 100nF, resistor:C1206
- added C1_2, C2_2, C3_2: 10uF, resistor:C1206
- added ENC_1, ENC_2, ENC_3: ENCODER_AS5045B, minebot_PDR:SSOP16
- added F5, F6, F7, F8: 60VDC 3A, minebot_PDR:OMNI_BLOCK
- added F9: 60VDC 5A, minebot_PDR:OMNI_BLOCK
- added MAIN_1, MAIN_2, MAIN_3, SUB_1, SUB_2, SUB_3: (no value), pinhead:1X06
- added R10, R9: 500, resistor:R1206
- added R5, R6, R7: 1100, resistor:R1206
- added R8: 150, resistor:R1206
- added RVP_2, RVP_3: 25V, diode:SMC
- added RVP_4, RVP_5, RVP_6: 5V, diode:SMC
- added RVP_7, RVP_8: 15V, diode:SMC
- F1: value 24V_20A -> 100VDC 20A; device fuse:TE5 -> minebot_PDR:NANO
- F2: value 24V, 15A -> 60VDC 5A; device fuse:TE5 -> minebot_PDR:OMNI_BLOCK
- F3: value 12V_2A -> 60VDC 5A; device fuse:TE5 -> minebot_PDR:OMNI_BLOCK
- F4: value 5V_1A -> 60VDC 5A; device fuse:TE5 -> minebot_PDR:OMNI_BLOCK
- R2: value 1100 -> 150
- RVP_1: value (none) -> 25V
- moved F1 600.6 mm to (-167.1, -516.8), turned to 0 degrees
- moved R4 516.0 mm to (-171.1, -465.5), turned to 0 degrees
- moved R2 515.9 mm to (-171.1, -453.3), turned to 0 degrees
- moved RPI_OUT 424.2 mm to (-91.2, -364.5), turned to 0 degrees
- moved F4 403.1 mm to (-79.4, -342.6)
- moved F3 330.6 mm to (-79.4, -297.1)
- moved F2 294.4 mm to (-89.9, -211.8), turned to 0 degrees
- moved RVP_1 213.6 mm to (-74.2, -135.4), turned to 0 degrees
- renumbered 12V_TEST1 to 12V_TEST, 24V_TEST2 to 24V_TEST
Connections:
- removed net 24V_REG_MOTOR: 24V_TEST.TP, F2.2, R2.1, STEPPER_OUT.1
- removed net N$7: C6.2, F4.1, TVS_5.1, VREG_2.3
- new net 12V_REG1: 12V_5A.1, F9.VIN-, R9.1
- new net 12V_REG2: 12V_3A.1, F8.VIN-, R10.1
- new net 5V_REG1: F5.VIN-, R2.2, RPI_OUT.1
- new net 5V_REG2: 5V_OUT.1, F6.VIN-, R4.2
- new net 5V_REG3: 5V_RAIL.1, 5V_RAIL.3, 5V_RAIL.5, 5V_RAIL.7, 5V_RAIL.9, F7.VIN-, R8.2
- new net A_1: ENC_1.3, SUB_1.3
- new net A_2: ENC_2.3, SUB_2.3
- new net A_3: ENC_3.3, SUB_3.3
- new net B_1: ENC_1.4, SUB_1.4
- new net B_2: ENC_2.4, SUB_2.4
- new net B_3: ENC_3.4, SUB_3.4
- new net CLK_1: ENC_1.10, MAIN_1.4
- new net CLK_2: ENC_2.10, MAIN_2.4
- new net CLK_3: ENC_3.10, MAIN_3.4
- new net CSN_1: ENC_1.11, MAIN_1.3
- new net CSN_2: ENC_2.11, MAIN_2.3
- new net CSN_3: ENC_3.11, MAIN_3.3
- new net DO_1: ENC_1.9, MAIN_1.5
- new net DO_2: ENC_2.9, MAIN_2.5
- new net DO_3: ENC_3.9, MAIN_3.5
- new net GND_1: C1_1.2, C1_2.2, ENC_1.7, MAIN_1.2
- new net GND_2: C2_1.2, C2_2.2, ENC_2.7, MAIN_2.2
- new net GND_3: C3_1.2, C3_2.2, ENC_3.7, MAIN_3.2
- new net I_1: ENC_1.6, SUB_1.5
- new net I_2: ENC_2.6, SUB_2.5
- new net I_3: ENC_3.6, SUB_3.5
- new net MAG_DEC_N_1: ENC_1.2, SUB_1.2
- new net MAG_DEC_N_2: ENC_2.2, SUB_2.2
- new net MAG_DEC_N_3: ENC_3.2, SUB_3.2
- new net MAG_INC_N_1: ENC_1.1, SUB_1.1
- new net MAG_INC_N_2: ENC_2.1, SUB_2.1
- new net MAG_INC_N_3: ENC_3.1, SUB_3.1
- new net N$12: F2.VIN-, R5.1, STEPPER_OUT_1.1
- new net N$14: F3.VIN+, RVP_2.C
- new net N$16: R6.2, STEPPER_2.A
- new net N$18: F3.VIN-, R6.1, STEPPER_OUT_2.1
- new net N$22: F4.VIN+, RVP_3.C
- new net N$24: R7.2, STEPPER_3.A
- new net N$25: F4.VIN-, R7.1, STEPPER_OUT_3.1
- new net N$28: F6.VIN+, RVP_5.C
- new net N$29: 12V_3A_.A, R10.2
- new net N$32: F7.VIN+, RVP_6.C
- new net N$35: F8.VIN+, RVP_7.C
- new net N$36: F9.VIN+, RVP_8.C
- new net N$4: C1_2.1, ENC_1.15
- new net N$5: F2.VIN+, RVP_1.C
- new net N$6: C3_2.1, ENC_3.15
- new net PDIO_1: ENC_1.8, SUB_1.6
- new net PDIO_2: ENC_2.8, SUB_2.6
- new net PDIO_3: ENC_3.8, SUB_3.6
- new net PWM_1: ENC_1.12, MAIN_1.6
- new net PWM_2: ENC_2.12, MAIN_2.6
- new net PWM_3: ENC_3.12, MAIN_3.6
- new net VIN_1: C1_1.1, ENC_1.16, MAIN_1.1
- new net VIN_2: C2_1.1, ENC_2.16, MAIN_2.1
- new net VIN_3: C3_1.1, ENC_3.16, MAIN_3.1
- net 12V_REG: now also C4.2, RVP_7.A, RVP_8.A, TVS_3.1, VREG_1.3; no longer DCMOTOR_OUT.1, R3.1, TVS_4.C
- net 24V_REG: now also 24V_TEST.TP, F1.VIN-, R1.1, RVP_1.A, RVP_2.A, RVP_3.A; no longer F2.1, RVP_1.C
- net 5V_REG: now also C6.2, RVP_4.A, RVP_5.A, RVP_6.A, TVS_5.1, VREG_2.3; no longer AUX.1, GPS_OUT.1, R4.2, RPI_OUT.1, TVS_6.C
- net GND: now also 12V_3A.2, 12V_3A_.C, 12V_5A.2, 12V_5A_.C, 5V_OUT.2, 5V_RAIL.10, 5V_RAIL.2, 5V_RAIL.4, 5V_RAIL.6, 5V_RAIL.8, OUT_5V.C, RAIL_5V.C, RPI_5V.C, STEPPER_1.C, STEPPER_2.C, STEPPER_3.C, STEPPER_OUT_1.2, STEPPER_OUT_2.2, STEPPER_OUT_3.2; no longer 12V.C, 5V.C, AUX.2, DCMOTOR_OUT.2, GPS_OUT.2, STEPPER.C, STEPPER_OUT.2
- net N$10: now also R2.1, RPI_5V.A; no longer C4.2, F3.1, TVS_3.1, VREG_1.3
- net N$11: now also R8.1, RAIL_5V.A; no longer F4.2, TVS_6.A
- net N$17: now also 12V_5A_.A, R9.2; no longer F3.2, TVS_4.A
- net N$2: now also C2_2.1, ENC_2.15; no longer 12V.A, R3.2
- net N$20: now also OUT_5V.A; no longer 5V.A
- net N$3: now also F1.VIN+; no longer F1.1
- net N$8: now also F5.VIN+, RVP_4.C; no longer R2.2, STEPPER.A
- net N$9: now also R5.2, STEPPER_1.A; no longer F1.2, R1.1, RVP_1.A
Routing:
- net GND: track 212.7 -> 120.6 mm
- net 24V_REG_MOTOR: track 64.8 -> 0.00 mm, vias 1 -> 0
- net 5V_REG: track 92.2 -> 28.0 mm, vias 1 -> 0
- net 12V_REG: track 76.3 -> 30.6 mm, vias 1 -> 0
- net N$9: track 45.5 -> 0.00 mm, vias 2 -> 0
- net N$10: track 31.9 -> 0.00 mm
- net N$7: track 31.9 -> 0.00 mm
- net N$3: track 27.7 -> 7.36 mm
- net 24V_REG: track 79.2 -> 95.2 mm, vias 2 -> 3
- net N$17: track 8.31 -> 0.00 mm
- net N$11: track 8.27 -> 0.00 mm
- net N$20: track 3.31 -> 0.00 mm
- net N$2: track 3.31 -> 0.00 mm
- net N$8: track 3.31 -> 0.00 mm

Commit message: schematic finalized
Parts:
- removed 5V_OUT: C-GRID-02-70543, con-molex:70543-02
- removed F9: 60VDC 5A, minebot_PDR:OMNI_BLOCK
- removed OUT_5V: GREEN, led:SML1206
- removed RVP_5: 5V, diode:SMC
- added 12V_TEST_2: TPPAD1-13, testpad:P1-13
- added C7, C8: 10uF, resistor:C1206
- added R3: 1100, resistor:R1206
- added TVS_1: 26V, POWER_DISTRO:DO-214AC
- added VREG_3: LM1084ISX-5.0, POWER_DISTRO:TO-263-3
- 5V_RAIL: value 5v -> 5V 2A
- F8: value 60VDC 3A -> 60VDC 2A
- R10, R9: value 500 -> 150
- R2, R4: value 150 -> 1100
- R5, R6: value 1100 -> 500
- R7: value 1100 -> 365_1%
- R8: value 150 -> 121_1%
- TVS_2: value 26V -> 16V
- VREG_1: value 12V -> 12V 3A
- VREG_2: value 5V -> 12V 3A
- moved RVP_8 505.8 mm to (52.1, 11.6), turned to 180 degrees
- moved F6 448.8 mm to (65.5, 12.2)
- moved R7 442.1 mm to (-171.1, -789.8)
- moved R5 390.1 mm to (-171.1, -502.0)
- moved R2 343.4 mm to (-66.4, -126.2)
- moved R8 318.4 mm to (-171.1, -796.0)
- moved F7 253.1 mm to (-89.9, -192.3)
- moved R6 195.9 mm to (-171.1, -489.8)
- moved F8 184.7 mm to (-100.3, -445.1)
- moved R4 133.6 mm to (-97.7, -353.8)
- moved F5 68.5 mm to (-89.9, -260.7)
- moved TVS_2 51.4 mm to (40.6, 5.59), turned to 0 degrees
- moved C5 43.0 mm to (48.9, 17.9), turned to 0 degrees
- moved R9 36.6 mm to (-171.1, -453.3)
- moved VREG_2 35.3 mm to (56.8, 25.8), turned to 0 degrees
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- renumbered 12V_3A to 12V_3A_1, 12V_3A_ to 12V_3A_1_, 12V_5A to 12V_3A_2, 12V_5A_ to 12V_3A_2_, 12V_TEST to 12V_TEST_1, TVS_5 to TVS_4
Connections:
- removed net 12V_REG2: 12V_3A_1.1, F8.VIN-, R10.1
- removed net 5V_REG2: 5V_OUT.1, F6.VIN-, R4.2
- removed net N$28: F6.VIN+, RVP_5.C
- removed net N$35: F8.VIN+, RVP_7.C
- new net N$13: F5.VIN+, RVP_7.C
- new net N$15: R7.1, R8.2, VREG_3.1, VREG_3.4
- new net N$7: 12V_TEST_1.TP, C4.2, RVP_7.A, TVS_2.1, VREG_1.3
- net 12V_REG: now also 12V_TEST_2.TP, C6.2, VREG_2.3; no longer 12V_TEST_1.TP, C4.2, RVP_7.A, VREG_1.3
- net 12V_REG1: now also F6.VIN-, R6.1; no longer F9.VIN-, R9.1
- net 24V_REG: now also C7.2, TVS_1.1, VREG_3.3; no longer TVS_2.1
- net 5V_REG: now also C8.2, R8.1, VREG_3.2; no longer C6.2, RVP_5.A, VREG_2.3
- net 5V_REG1: now also F7.VIN-, R9.2; no longer F5.VIN-, R2.2
- net 5V_REG3: now also F8.VIN-, R10.2; no longer F7.VIN-, R8.2
- net GND: now also C7.1, C8.1, R7.2, TVS_1.2; no longer 5V_OUT.2, OUT_5V.C
- net N$10: now also R9.1; no longer R2.1
- net N$11: now also R10.1; no longer R8.1
- net N$12: now also R2.1; no longer R5.1
- net N$16: now also R3.2; no longer R6.2
- net N$17: now also R6.2; no longer R9.2
- net N$18: now also R3.1; no longer R6.1
- net N$20: now also 12V_3A_1.1, F5.VIN-, R5.1; no longer OUT_5V.A, R4.1
- net N$24: now also R4.2; no longer R7.2
- net N$25: now also R4.1; no longer R7.1
- net N$29: now also R5.2; no longer R10.2
- net N$32: now also F8.VIN+; no longer F7.VIN+
- net N$36: now also F6.VIN+; no longer F9.VIN+
- net N$8: now also F7.VIN+; no longer F5.VIN+
- net N$9: now also R2.2; no longer R5.2
Routing:
- net GND: track 120.6 -> 70.7 mm, vias 25 -> 19
- net 12V_REG: track 30.6 -> 0.00 mm
- net 24V_REG: track 95.2 -> 67.8 mm
