File: task_12_PDS PCB/Power_Distro_Board.sch (EAGLE design)
At the start: 35 parts

Commit message: PCB sch done, added another lib called minebot_PDR.lbr
Parts:
- removed 12V, 5V, STEPPER: GREEN, led:LEDSML1206
- removed 12V_TEST1: TPPAD1-13, testpad:TPPAD1-13
- removed AUX, GPS_OUT: C-GRID-02-70543, con-molex:C-GRID-02-70543
- removed DCMOTOR_OUT, STEPPER_OUT: 5566-2, con-molex:5566-2
- removed R3: 500, resistor:R-US_R1206
- removed TVS_4: 16V, diode:SCHOTTKY-DIODESMC
- removed TVS_6: 5V, diode:SCHOTTKY-DIODESMC
- added 12V_3A, 12V_5A, STEPPER_OUT_1, STEPPER_OUT_2, STEPPER_OUT_3: 5566-2, con-molex:5566-2
- added 12V_3A_, 12V_5A_, OUT_5V, RAIL_5V, RPI_5V, STEPPER_1, STEPPER_2, STEPPER_3: GREEN, led:LEDSML1206
- added 12V_TEST: TPPAD1-13, testpad:TPPAD1-13
- added 5V_OUT: C-GRID-02-70543, con-molex:C-GRID-02-70543
- added 5V_RAIL: 5v, pinhead:PINHD-2X5
- added C1_1, C2_1, C3_1: 100nF, resistor:C-EUC1206
- added C1_2, C2_2, C3_2: 10uF, resistor:C-EUC1206
- added ENC_1, ENC_2, ENC_3: ENCODER_AS5045B, minebot_PDR:ENCODER_AS5045B
- added F5, F6, F7, F8: 60VDC 3A, minebot_PDR:LITTLEFUSE0154
- added F9: 60VDC 5A, minebot_PDR:LITTLEFUSE0154
- added MAIN_1, MAIN_2, MAIN_3, SUB_1, SUB_2, SUB_3: (no value), pinhead:PINHD-1X6
- added R10, R9: 500, resistor:R-US_R1206
- added R5, R6, R7: 1100, resistor:R-US_R1206
- added R8: 150, resistor:R-US_R1206
- added RVP_2, RVP_3: 25V, diode:SCHOTTKY-DIODESMC
- added RVP_4, RVP_5, RVP_6: 5V, diode:SCHOTTKY-DIODESMC
- added RVP_7, RVP_8: 15V, diode:SCHOTTKY-DIODESMC
- F1: value 24V_20A -> 100VDC 20A; device fuse:TE5 -> minebot_PDR:LITTLEFUSENANO463
- F2: value 24V, 15A -> 60VDC 5A; device fuse:TE5 -> minebot_PDR:LITTLEFUSE0154
- F3: value 12V_2A -> 60VDC 5A; device fuse:TE5 -> minebot_PDR:LITTLEFUSE0154
- F4: value 5V_1A -> 60VDC 5A; device fuse:TE5 -> minebot_PDR:LITTLEFUSE0154
- R2: value 1100 -> 150
- RVP_1: value (none) -> 25V
- renumbered 24V_TEST2 to 24V_TEST
Connections:
- removed net 24V_REG_MOTOR: 24V_TEST.TP, F2.2, R2.1, STEPPER_OUT-1.S
- removed net N$7: C6.2, F4.1, TVS_5.C, VREG_2.OUT
- new net 12V_REG1: 12V_5A-1.S, F9.VIN-, R9.1
- new net 12V_REG2: 12V_3A-1.S, F8.VIN-, R10.1
- new net 5V_REG1: F5.VIN-, R2.2, RPI_OUT-1.S
- new net 5V_REG2: 5V_OUT-1.S, F6.VIN-, R4.2
- new net 5V_REG3: 5V_RAIL.1, 5V_RAIL.3, 5V_RAIL.5, 5V_RAIL.7, 5V_RAIL.9, F7.VIN-, R8.2
- new net A_1: ENC_1.A, SUB_1.3
- new net A_2: ENC_2.A, SUB_2.3
- new net A_3: ENC_3.A, SUB_3.3
- new net B_1: ENC_1.B, SUB_1.4
- new net B_2: ENC_2.B, SUB_2.4
- new net B_3: ENC_3.B, SUB_3.4
- new net CLK_1: ENC_1.CLK, MAIN_1.4
- new net CLK_2: ENC_2.CLK, MAIN_2.4
- new net CLK_3: ENC_3.CLK, MAIN_3.4
- new net CSN_1: ENC_1.CSN, MAIN_1.3
- new net CSN_2: ENC_2.CSN, MAIN_2.3
- new net CSN_3: ENC_3.CSN, MAIN_3.3
- new net DO_1: ENC_1.DO, MAIN_1.5
- new net DO_2: ENC_2.DO, MAIN_2.5
- new net DO_3: ENC_3.DO, MAIN_3.5
- new net GND_1: C1_1.2, C1_2.2, ENC_1.VSS, MAIN_1.2
- new net GND_2: C2_1.2, C2_2.2, ENC_2.VSS, MAIN_2.2
- new net GND_3: C3_1.2, C3_2.2, ENC_3.VSS, MAIN_3.2
- new net I_1: ENC_1.I, SUB_1.5
- new net I_2: ENC_2.I, SUB_2.5
- new net I_3: ENC_3.I, SUB_3.5
- new net MAG_DEC_N_1: ENC_1.MAG_DEC_N, SUB_1.2
- new net MAG_DEC_N_2: ENC_2.MAG_DEC_N, SUB_2.2
- new net MAG_DEC_N_3: ENC_3.MAG_DEC_N, SUB_3.2
- new net MAG_INC_N_1: ENC_1.MAG_INC_N, SUB_1.1
- new net MAG_INC_N_2: ENC_2.MAG_INC_N, SUB_2.1
- new net MAG_INC_N_3: ENC_3.MAG_INC_N, SUB_3.1
- new net N$12: F2.VIN-, R5.1, STEPPER_OUT_1-1.S
- new net N$14: F3.VIN+, RVP_2.C
- new net N$16: R6.2, STEPPER_2.A
- new net N$18: F3.VIN-, R6.1, STEPPER_OUT_2-1.S
- new net N$22: F4.VIN+, RVP_3.C
- new net N$24: R7.2, STEPPER_3.A
- new net N$25: F4.VIN-, R7.1, STEPPER_OUT_3-1.S
- new net N$28: F6.VIN+, RVP_5.C
- new net N$29: 12V_3A_.A, R10.2
- new net N$32: F7.VIN+, RVP_6.C
- new net N$35: F8.VIN+, RVP_7.C
- new net N$36: F9.VIN+, RVP_8.C
- new net N$4: C1_2.1, ENC_1.VDD3V3
- new net N$5: F2.VIN+, RVP_1.C
- new net N$6: C3_2.1, ENC_3.VDD3V3
- new net PDIO_1: ENC_1.PDIO, SUB_1.6
- new net PDIO_2: ENC_2.PDIO, SUB_2.6
- new net PDIO_3: ENC_3.PDIO, SUB_3.6
- new net PWM_1: ENC_1.PWM, MAIN_1.6
- new net PWM_2: ENC_2.PWM, MAIN_2.6
- new net PWM_3: ENC_3.PWM, MAIN_3.6
- new net VIN_1: C1_1.1, ENC_1.VDD5V, MAIN_1.1
- new net VIN_2: C2_1.1, ENC_2.VDD5V, MAIN_2.1
- new net VIN_3: C3_1.1, ENC_3.VDD5V, MAIN_3.1
- net 12V_REG: now also 12V_TEST.TP, C4.2, RVP_7.A, RVP_8.A, TVS_3.C, VREG_1.OUT; no longer 12V_TEST1.TP, DCMOTOR_OUT-1.S, R3.1, TVS_4.C
- net 24V_REG: now also 24V_TEST.TP, F1.VIN-, R1.1, RVP_1.A, RVP_2.A, RVP_3.A; no longer F2.1, RVP_1.C
- net 5V_REG: now also C6.2, RVP_4.A, RVP_5.A, RVP_6.A, TVS_5.C, VREG_2.OUT; no longer AUX-1.S, GPS_OUT-1.S, R4.2, RPI_OUT-1.S, TVS_6.C
- net GND: now also 12V_3A-2.S, 12V_3A_.C, 12V_5A-2.S, 12V_5A_.C, 5V_OUT-2.S, 5V_RAIL.10, 5V_RAIL.2, 5V_RAIL.4, 5V_RAIL.6, 5V_RAIL.8, OUT_5V.C, RAIL_5V.C, RPI_5V.C, STEPPER_1.C, STEPPER_2.C, STEPPER_3.C, STEPPER_OUT_1-2.S, STEPPER_OUT_2-2.S, STEPPER_OUT_3-2.S; no longer 12V.C, 5V.C, AUX-2.S, DCMOTOR_OUT-2.S, GPS_OUT-2.S, STEPPER.C, STEPPER_OUT-2.S
- net N$10: now also R2.1, RPI_5V.A; no longer C4.2, F3.1, TVS_3.C, VREG_1.OUT
- net N$11: now also R8.1, RAIL_5V.A; no longer F4.2, TVS_6.A
- net N$17: now also 12V_5A_.A, R9.2; no longer F3.2, TVS_4.A
- net N$2: now also C2_2.1, ENC_2.VDD3V3; no longer 12V.A, R3.2
- net N$20: now also OUT_5V.A; no longer 5V.A
- net N$3: now also F1.VIN+; no longer F1.1
- net N$8: now also F5.VIN+, RVP_4.C; no longer R2.2, STEPPER.A
- net N$9: now also R5.2, STEPPER_1.A; no longer F1.2, R1.1, RVP_1.A
Other:
- note added: "**These 3 encoder PCBs will be cut out of the main board"
- note added: "Rotary Encoder PCB 1"
- note added: "Rotary Encoder PCB 2"
- note added: "Rotary Encoder PCB 3"
- moved on the sheet: C1, C3, C4, PWR_IN-1, PWR_IN-2, R2, R4, RPI_OUT-1, RPI_OUT-2, RVP_1, TVS_3, VREG_1

Commit message: schematic finalized
Parts:
- removed 12V_5A: 5566-2, con-molex:5566-2
- removed 12V_5A_, OUT_5V: GREEN, led:LEDSML1206
- removed 12V_TEST: TPPAD1-13, testpad:TPPAD1-13
- removed 5V_OUT: C-GRID-02-70543, con-molex:C-GRID-02-70543
- removed F9: 60VDC 5A, minebot_PDR:LITTLEFUSE0154
- removed RVP_5: 5V, diode:SCHOTTKY-DIODESMC
- removed TVS_5: 5V, POWER_DISTRO:SMAJ5.0_TVSSMA
- added 12V_3A_2: 5566-2, con-molex:5566-2
- added 12V_3A_2_: GREEN, led:LEDSML1206
- added 12V_TEST_1, 12V_TEST_2: TPPAD1-13, testpad:TPPAD1-13
- added C7, C8: 10uF, resistor:C-EUC1206
- added R3: 1100, resistor:R-US_R1206
- added TVS_1: 26V, POWER_DISTRO:SMAJ26A_TVSSMA
- added TVS_4: 5V, POWER_DISTRO:SMAJ5.0_TVSSMA
- added VREG_3: LM1084ISX-5.0, POWER_DISTRO:LM1084ISX-5.0
- 5V_RAIL: value 5v -> 5V 2A
- F8: value 60VDC 3A -> 60VDC 2A
- R10, R9: value 500 -> 150
- R2, R4: value 150 -> 1100
- R5, R6: value 1100 -> 500
- R7: value 1100 -> 365_1%
- R8: value 150 -> 121_1%
- TVS_2: value 26V -> 16V; device POWER_DISTRO:SMAJ26A_TVSSMA -> POWER_DISTRO:PRSMA16_TVS
- VREG_1: value 12V -> 12V 3A; device POWER_DISTRO:HIGH-CURRENT_REGSMA -> POWER_DISTRO:MIC29300-12WUSMA
- VREG_2: value 5V -> 12V 3A; device POWER_DISTRO:HIGH-CURRENT_REGSMA -> POWER_DISTRO:MIC29300-12WUSMA
- renumbered 12V_3A to 12V_3A_1, 12V_3A_ to 12V_3A_1_
Connections:
- removed net 12V_REG2: 12V_3A_1-1.S, F8.VIN-, R10.1
- removed net 5V_REG2: 5V_OUT-1.S, F6.VIN-, R4.2
- removed net N$28: F6.VIN+, RVP_5.C
- removed net N$35: F8.VIN+, RVP_7.C
- new net N$13: F5.VIN+, RVP_7.C
- new net N$15: R7.1, R8.2, VREG_3.GND
- new net N$7: 12V_TEST_1.TP, C4.2, RVP_7.A, TVS_2.CATHODE, VREG_1.OUT
- net 12V_REG: now also 12V_TEST_2.TP, C6.2, TVS_3.CATHODE, VREG_2.OUT; no longer 12V_TEST.TP, C4.2, RVP_7.A, TVS_3.C, VREG_1.OUT
- net 12V_REG1: now also 12V_3A_2-1.S, F6.VIN-, R6.1; no longer 12V_5A-1.S, F9.VIN-, R9.1
- net 24V_REG: now also C7.2, TVS_1.CATHODE, VREG_3.IN; no longer TVS_2.C
- net 5V_REG: now also C8.2, R8.1, TVS_4.CATHODE, VREG_3.OUT; no longer C6.2, RVP_5.A, TVS_5.C, VREG_2.OUT
- net 5V_REG1: now also F7.VIN-, R9.2; no longer F5.VIN-, R2.2
- net 5V_REG3: now also F8.VIN-, R10.2; no longer F7.VIN-, R8.2
- net GND: now also 12V_3A_2-2.S, 12V_3A_2_.C, C7.1, C8.1, R7.2, TVS_1.ANODE, TVS_2.ANODE, TVS_3.ANODE, TVS_4.ANODE; no longer 12V_5A-2.S, 12V_5A_.C, 5V_OUT-2.S, OUT_5V.C, TVS_2.A, TVS_3.A, TVS_5.A
- net N$10: now also R9.1; no longer R2.1
- net N$11: now also R10.1; no longer R8.1
- net N$12: now also R2.1; no longer R5.1
- net N$16: now also R3.2; no longer R6.2
- net N$17: now also 12V_3A_2_.A, R6.2; no longer 12V_5A_.A, R9.2
- net N$18: now also R3.1; no longer R6.1
- net N$20: now also 12V_3A_1-1.S, F5.VIN-, R5.1; no longer OUT_5V.A, R4.1
- net N$24: now also R4.2; no longer R7.2
- net N$25: now also R4.1; no longer R7.1
- net N$29: now also R5.2; no longer R10.2
- net N$32: now also F8.VIN+; no longer F7.VIN+
- net N$36: now also F6.VIN+; no longer F9.VIN+
- net N$8: now also F7.VIN+; no longer F5.VIN+
- net N$9: now also R2.2; no longer R5.2
Other:
- note added: "**The ERC will say that there are no pins on net 12V_REG3, which I have not been able to find anywhere. It is not used anywhere too, I think it's a bug in EAGLE."
- moved on the sheet: 5V_TEST, C3, C4, C5, C6, F5, F6, F7, F8, R10, R2, R4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
