File: task_12_PDS PCB/Power_Distro_Board_V2.brd (EAGLE design)
At the start: 63.5 x 63.6 mm, 75 parts

Commit message: Gantry Code updated for DC motor and driver
Parts:
- removed R7: 365_1%, resistor:R1206
- removed R8: 121_1%, resistor:R1206
- removed RVP_4, RVP_6: 5V, diode:SMC
- removed TVS_4: 5V, POWER_DISTRO:DO-214AC
- removed VREG_3: LM1084ISX-5.0, POWER_DISTRO:TO-263-3
- added 2.5A, 5A: POLOLU_5VREG, POWER_DISTRO:SIP5
- added 5V_TEST1: TPPAD1-13, testpad:P1-13
- added C9: 10uF, resistor:C1206
- added EN2.5, EN5, PG2.5, PG5: MOUNT-PAD-ROUND2.8, holes:2,8-PAD
Connections:
- new net N$21: 2.5A.PG, PG2.5.B2,8
- new net N$23: 2.5A.EN, EN2.5.B2,8
- net 24V_REG: now also 2.5A.VIN, 5A.VIN; no longer VREG_3.3
- net 5V_REG: now also 2.5A.VOUT; no longer R8.1, RVP_4.A, RVP_6.A, TVS_4.1, VREG_3.2
- net GND: now also 2.5A.GND, 5A.GND, C9.1; no longer R7.2, TVS_4.2
- net N$15: now also 5A.EN, EN5.B2,8; no longer R7.1, R8.2, VREG_3.1, VREG_3.4
- net N$32: now also 5A.VOUT, 5V_TEST1.TP, C9.2; no longer RVP_6.C
- net N$8: now also 5A.PG, PG5.B2,8; no longer F7.VIN+, RVP_4.C
Routing:
- net 5V_REG: track 27.5 -> 0.00 mm
