File: task_12_PDS PCB/Power_Distro_Board_V2.brd (EAGLE design)
At the start: 63.5 x 63.6 mm, 80 parts

Commit message: PDB Board Updates
Parts:
- removed C2_1, C3_1: 100nF, resistor:C1206
- removed C2_2, C3_2: 10uF, resistor:C1206
- removed EN2.1, EN2.2, EN2.5, EN5, PG2.5, PG5: MOUNT-PAD-ROUND2.8, holes:2,8-PAD
- removed ENC_2, ENC_3: ENCODER_AS5045B, minebot_PDR:SSOP16
- removed MAIN_2, MAIN_3, SUB_2, SUB_3: (no value), pinhead:1X06
- added EN1, EN2, ENABLE1, ENABLE2, PG1, PG2: TPPAD1-13, testpad:P1-13
- F1: value 100VDC 20A -> 60VDC 50A
- F2, F3, F4, F6, F7: device minebot_PDR:OMNI_BLOCK -> resistor:R1206W
- F5: value 60VDC 3A -> 60VDC 20A; device minebot_PDR:OMNI_BLOCK -> resistor:R1206W
- F8: value 60VDC 5A -> 60VDC 3A; device minebot_PDR:OMNI_BLOCK -> resistor:R1206W
- F9: value 60VDC 20A -> 60VDC 5A; device minebot_PDR:OMNI_BLOCK -> resistor:R1206W
- R2, R3, R4, R7: value 500 -> 470
- RVP_1, RVP_2, RVP_3, RVP_4: value 13V -> 15V; device diode:SMC -> diode:TO220ACS
- TVS_1: value 26V -> 16V
- moved F6 1659.2 mm to (-169.0, -1463.7)
- moved F9 1571.3 mm to (-169.0, -1476.1)
- moved RVP_4 1391.8 mm to (-2.54, -1285.4)
- moved F7 1280.1 mm to (-169.0, -1469.9)
- moved F2 1219.0 mm to (-169.0, -1428.2)
- moved F5 1199.3 mm to (-169.0, -1457.5)
- moved F3 1151.4 mm to (-169.0, -1445.0)
- moved F4 1112.2 mm to (-169.0, -1451.2)
- moved RVP_1 1099.0 mm to (-2.54, -1232.0)
- moved F8 1039.5 mm to (-169.0, -1482.3)
- moved RVP_2 955.6 mm to (-2.54, -1249.8)
- moved RVP_3 927.9 mm to (-2.54, -1267.6)
- renumbered U$1 to 24V_REG1, U$2 to 24V_REG
Connections:
- removed net A_2: ENC_2.3, SUB_2.3
- removed net A_3: ENC_3.3, SUB_3.3
- removed net B_2: ENC_2.4, SUB_2.4
- removed net B_3: ENC_3.4, SUB_3.4
- removed net CLK_2: ENC_2.10, MAIN_2.4
- removed net CLK_3: ENC_3.10, MAIN_3.4
- removed net CSN_2: ENC_2.11, MAIN_2.3
- removed net CSN_3: ENC_3.11, MAIN_3.3
- removed net DO_2: ENC_2.9, MAIN_2.5
- removed net DO_3: ENC_3.9, MAIN_3.5
- removed net GND_2: C2_1.2, C2_2.2, ENC_2.7, MAIN_2.2
- removed net GND_3: C3_1.2, C3_2.2, ENC_3.7, MAIN_3.2
- removed net I_2: ENC_2.6, SUB_2.5
- removed net I_3: ENC_3.6, SUB_3.5
- removed net MAG_DEC_N_2: ENC_2.2, SUB_2.2
- removed net MAG_DEC_N_3: ENC_3.2, SUB_3.2
- removed net MAG_INC_N_2: ENC_2.1, SUB_2.1
- removed net MAG_INC_N_3: ENC_3.1, SUB_3.1
- removed net N$21: 2.5A.PG, PG2.5.B2,8
- removed net N$23: 2.5A.EN, EN2.5.B2,8
- removed net PDIO_2: ENC_2.8, SUB_2.6
- removed net PDIO_3: ENC_3.8, SUB_3.6
- removed net PWM_2: ENC_2.12, MAIN_2.6
- removed net PWM_3: ENC_3.12, MAIN_3.6
- removed net VIN_2: C2_1.1, ENC_2.16, MAIN_2.1
- removed net VIN_3: C3_1.1, ENC_3.16, MAIN_3.1
- net 5V_REG: now also F8.1
- net 5V_REG1: now also F8.2; no longer F7.VIN-
- net 5V_REG3: now also F9.2; no longer F8.VIN-
- net N$12: now also F2.2; no longer F2.VIN-
- net N$13: now also F6.1; no longer F5.VIN+
- net N$14: now also F3.1; no longer F3.VIN+
- net N$15: now also EN2.TP; no longer EN5.B2,8
- net N$18: now also F3.2; no longer F3.VIN-
- net N$2: now also 2.5A.PG, PG1.TP; no longer C2_2.1, ENC_2.15
- net N$20: now also F6.2; no longer F5.VIN-
- net N$22: now also F4.1; no longer F4.VIN+
- net N$25: now also F4.2; no longer F4.VIN-
- net N$26: now also F5.1; no longer F9.VIN+
- net N$28: now also F5.2; no longer F9.VIN-
- net N$30: now also ENABLE1.TP; no longer EN2.1.B2,8
- net N$32: now also F9.1; no longer F8.VIN+
- net N$33: now also F7.1; no longer F6.VIN+
- net N$34: now also F7.2; no longer F6.VIN-
- net N$35: now also ENABLE2.TP; no longer EN2.2.B2,8
- net N$5: now also F2.1; no longer F2.VIN+
- net N$6: now also 2.5A.EN, EN1.TP; no longer C3_2.1, ENC_3.15
- net N$8: now also PG2.TP; no longer PG5.B2,8
