File: task_12_PDS PCB/Power_Distro_Board_V2.sch (EAGLE design)
At the start: 75 parts

Commit message: Gantry Code updated for DC motor and driver
Parts:
- removed R7: 365_1%, resistor:R-US_R1206
- removed R8: 121_1%, resistor:R-US_R1206
- removed RVP_4, RVP_6: 5V, diode:SCHOTTKY-DIODESMC
- removed TVS_4: 5V, POWER_DISTRO:SMAJ5.0_TVSSMA
- removed VREG_3: LM1084ISX-5.0, POWER_DISTRO:LM1084ISX-5.0
- added 2.5A, 5A: POLOLU_5VREG, POWER_DISTRO:POLOLU_5VREG
- added 5V_TEST1: TPPAD1-13, testpad:TPPAD1-13
- added C9: 10uF, resistor:C-EUC1206
- added EN2.5, EN5, PG2.5, PG5: MOUNT-PAD-ROUND2.8, holes:MOUNT-PAD-ROUND2.8
Connections:
- new net N$21: 2.5A.PG, PG2.5.MOUNT
- new net N$23: 2.5A.EN, EN2.5.MOUNT
- net 24V_REG: now also 2.5A.VIN, 5A.VIN; no longer VREG_3.IN
- net 5V_REG: now also 2.5A.VOUT; no longer R8.1, RVP_4.A, RVP_6.A, TVS_4.CATHODE, VREG_3.OUT
- net GND: now also 2.5A.GND, 5A.GND, C9.1; no longer R7.2, TVS_4.ANODE
- net N$15: now also 5A.EN, EN5.MOUNT; no longer R7.1, R8.2, VREG_3.GND
- net N$32: now also 5A.VOUT, 5V_TEST1.TP, C9.2; no longer RVP_6.C
- net N$8: now also 5A.PG, PG5.MOUNT; no longer F7.VIN+, RVP_4.C
Other:
- moved on the sheet: 5V_TEST, C7, C8
