File: task_12_PDS PCB/Power_Distro_Board_V3.brd (EAGLE design)
At the start: 63.5 x 63.6 mm, 70 parts

Commit message: PDB Board Updates
Parts:
- removed 24V_2A_1, 24V_2A_2: 5566-2, con-molex:5566-2
- removed 24V_2A_1_, 24V_2A_1_1: GREEN, led:SML1206
- removed 24V_REG, 24V_REG1: POLOLU_24VSTEPUP, POWER_DISTRO:2X4PIN_REG
- removed 24V_TEST_1, 24V_TEST_2: TPPAD1-13, testpad:P1-13
- removed C3, C4, C5, C6: 10uF, resistor:C1206
- removed EN2.1, EN2.2, EN2.5, EN5, PG2.5, PG5: MOUNT-PAD-ROUND2.8, holes:2,8-PAD
- added 12V_5, 12V_6: GREEN, led:SML1206
- added EN1, EN2, PG1, PG2: TPPAD1-13, testpad:P1-13
- added MOTOR_OUT_5, MOTOR_OUT_6: 5566-2, con-molex:5566-2
- added RVP_5, RVP_6: 15V, diode:TO220ACS
- F1: value 100VDC 20A -> 60VDC 50A
- F2, F3, F4: device minebot_PDR:OMNI_BLOCK -> resistor:R1206W
- F5, F6, F7: value 60VDC 3A -> 60VDC 20A; device minebot_PDR:OMNI_BLOCK -> resistor:R1206W
- F8: value 60VDC 5A -> 60VDC 3A; device minebot_PDR:OMNI_BLOCK -> resistor:R1206W
- F9: value 60VDC 20A -> 60VDC 5A; device minebot_PDR:OMNI_BLOCK -> resistor:R1206W
- R2, R3, R4, R7: value 500 -> 470
- R5, R6: value 1100 -> 470
- RVP_1, RVP_2, RVP_3, RVP_4: value 13V -> 15V; device diode:SMC -> diode:TO220ACS
- TVS_1: value 26V -> 16V
- moved 5V_TEST1 896.3 mm to (25.1, 12.1)
- moved C9 884.1 mm to (30.1, 10.4)
- moved 5A 878.6 mm to (29.2, 26.2)
- moved 2.5A 851.0 mm to (10.0, 26.0)
- moved SUB_1 747.9 mm to (29.6, 109.2), turned to 270 degrees
- moved MAIN_1 732.0 mm to (49.4, 102.4), turned to 270 degrees
- moved C1_2 701.6 mm to (44.5, 124.8)
- moved C1_1 691.3 mm to (46.0, 119.8), turned to 180 degrees
- moved ENC_1 674.3 mm to (45.1, 112.0)
- moved F1 614.4 mm to (15.5, 69.8), turned to 180 degrees
- moved R5 581.8 mm to (50.8, 35.8), turned to 90 degrees
- moved RAIL_5V 525.6 mm to (30.5, 2.54), turned to 180 degrees
- moved R10 524.3 mm to (30.2, 6.48)
- moved RPI_5V 495.8 mm to (11.6, 2.41), turned to 180 degrees
- moved R9 494.4 mm to (11.6, 6.22)
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Connections:
- removed net N$29: 24V_2A_1_.A, R5.2
- removed net N$30: 24V_REG1.ENABLE, EN2.1.B2,8
- removed net N$31: 24V_REG.VOUT1, 24V_REG.VOUT2, 24V_TEST_2.TP, C6.2
- removed net N$33: F6.VIN+
- removed net N$34: 24V_2A_2.1, F6.VIN-, R6.1
- removed net N$35: 24V_REG.ENABLE, EN2.2.B2,8
- new net N$2: 2.5A.PG, PG1.TP
- new net N$6: 2.5A.EN, EN1.TP
- net 12V_REG: now also RVP_5.A, RVP_6.A
- net 12V_REG_TVS: no longer 24V_REG.VIN1, 24V_REG.VIN2, 24V_REG1.VIN1, 24V_REG1.VIN2, C3.2, C5.2
- net 5V_REG: now also F8.1
- net 5V_REG1: now also F8.2; no longer F7.VIN-
- net 5V_REG3: now also F9.2; no longer F8.VIN-
- net GND: now also 12V_5.C, 12V_6.C, MOTOR_OUT_5.2, MOTOR_OUT_6.2; no longer 24V_2A_1.2, 24V_2A_1_.C, 24V_2A_1_1.C, 24V_2A_2.2, 24V_REG.GND1, 24V_REG.GND2, 24V_REG.GND3, 24V_REG.GND4, 24V_REG1.GND1, 24V_REG1.GND2, 24V_REG1.GND3, 24V_REG1.GND4, C3.1, C4.1, C5.1, C6.1
- net N$12: now also F2.2; no longer F2.VIN-
- net N$13: now also 12V_5.A, R6.2; no longer F5.VIN+
- net N$14: now also F3.1; no longer F3.VIN+
- net N$15: now also EN2.TP; no longer EN5.B2,8
- net N$17: now also F6.2, MOTOR_OUT_5.1, R6.1; no longer 24V_2A_1_1.A, R6.2
- net N$18: now also F3.2; no longer F3.VIN-
- net N$20: now also F7.1, RVP_6.C; no longer 24V_2A_1.1, F5.VIN-, R5.1
- net N$21: now also 12V_6.A, R7.2; no longer 2.5A.PG, PG2.5.B2,8
- net N$22: now also F4.1; no longer F4.VIN+
- net N$23: now also F7.2, MOTOR_OUT_6.1, R7.1; no longer 2.5A.EN, EN2.5.B2,8
- net N$25: now also F4.2; no longer F4.VIN-
- net N$26: now also F5.1; no longer F9.VIN+
- net N$27: now also R5.2; no longer R7.2
- net N$28: now also F5.2, R5.1; no longer F9.VIN-, R7.1
- net N$32: now also F9.1; no longer F8.VIN+
- net N$5: now also F2.1; no longer F2.VIN+
- net N$7: now also F6.1, RVP_5.C; no longer 24V_REG1.VOUT1, 24V_REG1.VOUT2, 24V_TEST_1.TP, C4.2
- net N$8: now also PG2.TP; no longer PG5.B2,8
Routing:
- net GND: track 70.7 -> 0.00 mm, vias 19 -> 0
- net 12V_REG: track 57.4 -> 0.00 mm, vias 3 -> 0
- net 12V_REG_TVS: track 10.4 -> 0.00 mm
- net N$3: track 7.36 -> 0.00 mm, vias 1 -> 0
- net N$1: track 3.31 -> 0.00 mm
Other:
- board size 63.5 x 63.6 mm -> 63.5 x 127 mm
