File: task_12_PDS PCB/Power_Distro_Board_V3.sch (EAGLE design)
At the start: 80 parts

Commit message: PDB Board Updates
Parts:
- removed 24V_2A_1, 24V_2A_2: 5566-2, con-molex:5566-2
- removed 24V_2A_1_, 24V_2A_1_1: GREEN, led:LEDSML1206
- removed 24V_TEST_1, 24V_TEST_2: TPPAD1-13, testpad:TPPAD1-13
- removed C2_1, C3_1: 100nF, resistor:C-EUC1206
- removed C2_2, C3, C3_2, C4, C5, C6: 10uF, resistor:C-EUC1206
- removed EN2.1, EN2.2, EN2.5, EN5, PG2.5, PG5: MOUNT-PAD-ROUND2.8, holes:MOUNT-PAD-ROUND2.8
- removed ENC_2, ENC_3: ENCODER_AS5045B, minebot_PDR:ENCODER_AS5045B
- removed MAIN_2, MAIN_3, SUB_2, SUB_3: (no value), pinhead:PINHD-1X6
- removed U$1, U$2: POLOLU_24VSTEPUP, POWER_DISTRO:POLOLU_24VSTEPUP
- added 12V_5, 12V_6: GREEN, led:LEDSML1206
- added EN1, EN2, PG1, PG2: TPPAD1-13, testpad:TPPAD1-13
- added MOTOR_OUT_5, MOTOR_OUT_6: 5566-2, con-molex:5566-2
- added RVP_5, RVP_6: 15V, diode:BYT08P
- F1: value 100VDC 20A -> 60VDC 50A
- F2, F3, F4: device minebot_PDR:LITTLEFUSE0154 -> resistor:R-EU_R1206W
- F5, F6, F7: value 60VDC 3A -> 60VDC 20A; device minebot_PDR:LITTLEFUSE0154 -> resistor:R-EU_R1206W
- F8: value 60VDC 5A -> 60VDC 3A; device minebot_PDR:LITTLEFUSE0154 -> resistor:R-EU_R1206W
- F9: value 60VDC 20A -> 60VDC 5A; device minebot_PDR:LITTLEFUSE0154 -> resistor:R-EU_R1206W
- R2, R3, R4, R7: value 500 -> 470
- R5, R6: value 1100 -> 470
- RVP_1, RVP_2, RVP_3, RVP_4: value 13V -> 15V; device diode:SCHOTTKY-DIODESMC -> diode:BYT08P
- TVS_1: value 26V -> 16V
Connections:
- removed net A_2: ENC_2.A, SUB_2.3
- removed net A_3: ENC_3.A, SUB_3.3
- removed net B_2: ENC_2.B, SUB_2.4
- removed net B_3: ENC_3.B, SUB_3.4
- removed net CLK_2: ENC_2.CLK, MAIN_2.4
- removed net CLK_3: ENC_3.CLK, MAIN_3.4
- removed net CSN_2: ENC_2.CSN, MAIN_2.3
- removed net CSN_3: ENC_3.CSN, MAIN_3.3
- removed net DO_2: ENC_2.DO, MAIN_2.5
- removed net DO_3: ENC_3.DO, MAIN_3.5
- removed net GND_2: C2_1.2, C2_2.2, ENC_2.VSS, MAIN_2.2
- removed net GND_3: C3_1.2, C3_2.2, ENC_3.VSS, MAIN_3.2
- removed net I_2: ENC_2.I, SUB_2.5
- removed net I_3: ENC_3.I, SUB_3.5
- removed net MAG_DEC_N_2: ENC_2.MAG_DEC_N, SUB_2.2
- removed net MAG_DEC_N_3: ENC_3.MAG_DEC_N, SUB_3.2
- removed net MAG_INC_N_2: ENC_2.MAG_INC_N, SUB_2.1
- removed net MAG_INC_N_3: ENC_3.MAG_INC_N, SUB_3.1
- removed net N$29: 24V_2A_1_.A, R5.2
- removed net N$30: EN2.1.MOUNT, U$1.ENABLE
- removed net N$31: 24V_TEST_2.TP, C6.2, U$2.VOUT
- removed net N$33: F6.VIN+
- removed net N$34: 24V_2A_2-1.S, F6.VIN-, R6.1
- removed net N$35: EN2.2.MOUNT, U$2.ENABLE
- removed net PDIO_2: ENC_2.PDIO, SUB_2.6
- removed net PDIO_3: ENC_3.PDIO, SUB_3.6
- removed net PWM_2: ENC_2.PWM, MAIN_2.6
- removed net PWM_3: ENC_3.PWM, MAIN_3.6
- removed net VIN_2: C2_1.1, ENC_2.VDD5V, MAIN_2.1
- removed net VIN_3: C3_1.1, ENC_3.VDD5V, MAIN_3.1
- net 12V_REG: now also RVP_5.A, RVP_6.A
- net 12V_REG_TVS: no longer C3.2, C5.2, U$1.VIN, U$2.VIN
- net 5V_REG: now also F8.1
- net 5V_REG1: now also F8.2; no longer F7.VIN-
- net 5V_REG3: now also F9.2; no longer F8.VIN-
- net GND: now also 12V_5.C, 12V_6.C, MOTOR_OUT_5-2.S, MOTOR_OUT_6-2.S; no longer 24V_2A_1-2.S, 24V_2A_1_.C, 24V_2A_1_1.C, 24V_2A_2-2.S, C3.1, C4.1, C5.1, C6.1, U$1.GND1, U$1.GND2, U$2.GND1, U$2.GND2
- net N$12: now also F2.2; no longer F2.VIN-
- net N$13: now also 12V_5.A, R6.2; no longer F5.VIN+
- net N$14: now also F3.1; no longer F3.VIN+
- net N$15: now also EN2.TP; no longer EN5.MOUNT
- net N$17: now also F6.2, MOTOR_OUT_5-1.S, R6.1; no longer 24V_2A_1_1.A, R6.2
- net N$18: now also F3.2; no longer F3.VIN-
- net N$2: now also 2.5A.PG, PG1.TP; no longer C2_2.1, ENC_2.VDD3V3
- net N$20: now also F7.1, RVP_6.C; no longer 24V_2A_1-1.S, F5.VIN-, R5.1
- net N$21: now also 12V_6.A, R7.2; no longer 2.5A.PG, PG2.5.MOUNT
- net N$22: now also F4.1; no longer F4.VIN+
- net N$23: now also F7.2, MOTOR_OUT_6-1.S, R7.1; no longer 2.5A.EN, EN2.5.MOUNT
- net N$25: now also F4.2; no longer F4.VIN-
- net N$26: now also F5.1; no longer F9.VIN+
- net N$27: now also R5.2; no longer R7.2
- net N$28: now also F5.2, R5.1; no longer F9.VIN-, R7.1
- net N$32: now also F9.1; no longer F8.VIN+
- net N$5: now also F2.1; no longer F2.VIN+
- net N$6: now also 2.5A.EN, EN1.TP; no longer C3_2.1, ENC_3.VDD3V3
- net N$7: now also F6.1, RVP_5.C; no longer 24V_TEST_1.TP, C4.2, U$1.VOUT
- net N$8: now also PG2.TP; no longer PG5.MOUNT
Other:
- note removed: "Rotary Encoder PCB 2"
- note removed: "Rotary Encoder PCB 3"
- moved on the sheet: 12V_1, 12V_2, 12V_3, 12V_4, MOTOR_OUT_1-1, MOTOR_OUT_1-2, MOTOR_OUT_2-1, MOTOR_OUT_2-2, MOTOR_OUT_3-1, MOTOR_OUT_3-2, MOTOR_OUT_4-1, MOTOR_OUT_4-2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
