File: task_12_PDS PCB/Power_Distro_Board_V4.brd (EAGLE design)
At the start: 63.5 x 127 mm, 70 parts, among them J1 22-27-2081-08

Commit message: Completed PDB Board
Parts:
- removed 12V_IN: 5566-2, con-molex:5566-2
- removed C3: (no value), resistor:C1206
- removed DRV880_1, DRV880_2: (no value), pinhead:1X08
- removed ENABLE: TPPAD1-13, testpad:P1-13
- removed J1: 22-27-2081-08, con-molex:6410-08
- removed STEPPER_1: 5566-4, con-molex:5566-4
- removed U$1: POLOLU_24VSTEPUP, POWER_DISTRO:2X4PIN_REG
- added C1_3: 100nF, resistor:C1206
- added C1_4: 10uF, resistor:C1206
- added ENC_2: ENCODER_AS5045B, minebot_PDR:SSOP16
- added MAIN_2, SUB_2: (no value), pinhead:1X06
- moved MAIN_1 2.88 mm to (57.1, 108.8)
- moved SUB_1 2.88 mm to (37.3, 109.0)
- moved C1_1 2.88 mm to (44.6, 113.4)
- moved C1_2 2.88 mm to (50.8, 113.3)
- moved ENC_1 2.88 mm to (46.9, 106.8)
- moved RVP_2 0.90 mm to (36.1, 77.1)
- moved RVP_1 0.89 mm to (36.2, 84.8)
- moved 12V_2 0.51 mm to (60.5, 69.1)
- moved 12V_3 0.38 mm to (60.6, 55.1)
- moved 12V_4 0.38 mm to (60.6, 40.5)
- moved 12V_5 0.13 mm to (60.8, 25.5)
Connections:
- removed net 24V_1: DRV880_2.1, U$1.VOUT1, U$1.VOUT2
- removed net A1: DRV880_2.6, STEPPER_1.4
- removed net A2: DRV880_2.5, STEPPER_1.3
- removed net B1: DRV880_2.3, STEPPER_1.1
- removed net B2: DRV880_2.4, STEPPER_1.2
- removed net DIR: DRV880_1.8, J1.2
- removed net EN: DRV880_1.1, J1.7
- removed net FAULT: DRV880_2.7, J1.8
- removed net M0: DRV880_1.3, J1.5
- removed net M1: DRV880_1.2, J1.6
- removed net N$30: 12V_IN.1, U$1.VIN1, U$1.VIN2
- removed net N$31: ENABLE.TP, U$1.ENABLE
- removed net SLEEP: DRV880_1.6, J1.4
- removed net STEP: DRV880_1.7, J1.3
- removed net TRQ0: DRV880_1.5
- removed net TRQ1: DRV880_1.4
- new net A_2: ENC_2.3, SUB_2.3
- new net B_2: ENC_2.4, SUB_2.4
- new net CLK_2: ENC_2.10, MAIN_2.4
- new net CSN_2: ENC_2.11, MAIN_2.3
- new net DO_2: ENC_2.9, MAIN_2.5
- new net GND_2: C1_3.2, C1_4.2, ENC_2.7, MAIN_2.2
- new net I_2: ENC_2.6, SUB_2.5
- new net MAG_DEC_N_2: ENC_2.2, SUB_2.2
- new net MAG_INC_N_2: ENC_2.1, SUB_2.1
- new net PDIO_2: ENC_2.8, SUB_2.6
- new net PWM_2: ENC_2.12, MAIN_2.6
- new net VIN_2: C1_3.1, ENC_2.16, MAIN_2.1
- net GND: no longer C3.1, DRV880_2.2, DRV880_2.8, J1.1, U$1.GND3, U$1.GND4
- net N$29: now also C1_4.1, ENC_2.15; no longer 12V_IN.2, U$1.GND1, U$1.GND2
Routing:
- net GND_2: track 115.6 -> 40.2 mm
- net VIN_2: track 0.00 -> 19.7 mm
- net PWM_2: track 0.00 -> 14.0 mm
- net N$29: track 0.00 -> 10.1 mm, vias 0 -> 2
- net MAG_INC_N_2: track 0.00 -> 9.35 mm
- net CSN_2: track 0.00 -> 9.03 mm
- net MAG_DEC_N_2: track 0.00 -> 8.49 mm
- net CLK_2: track 0.00 -> 8.17 mm
- net PDIO_2: track 0.00 -> 6.90 mm
- net DO_2: track 0.00 -> 6.87 mm
- net A_2: track 0.00 -> 6.81 mm
- net I_2: track 0.00 -> 6.39 mm
- net N$15: track 33.6 -> 27.5 mm, vias 0 -> 2
- net B_2: track 0.00 -> 6.03 mm
- net N$20: track 35.1 -> 30.4 mm
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Other:
- board size 63.5 x 127 mm -> 63.8 x 122 mm
- board text removed: "**NOTE : There will be 27 DRC overlap errors. Those are all vias within the GND pad of the 3 linear voltage regulators included. These are added on purpose, with thermals generated, will help with power dissipation to the ground plane at the bottom."

Commit message: PDB Final Updates
Parts:
- removed F1: 60VDC 50A, minebot_PDR:NANO
- added F10: 20V, 50A, POWER_DISTRO:NANO
- F2, F3, F4, F5, F6, F7, F8, F9: device resistor:R1206W -> resistor:M1206
- moved ENC_1 1.81 mm to (47.5, 108.5)
- moved ENC_2 1.52 mm to (15.5, 108.5)
- moved SUB_1 0.81 mm to (38.0, 108.5)
- moved MAIN_2 0.76 mm to (26.0, 108.5)
- moved C1_2 0.62 mm to (50.8, 113.9)
- moved SUB_2 0.55 mm to (5.00, 108.5)
- moved C1_1 0.52 mm to (44.7, 113.9)
- moved MAIN_1 0.37 mm to (57.0, 108.5)
Connections:
- net 12V_REG: now also F10.P$1; no longer F1.VIN-
- net N$3: now also F10.P$2; no longer F1.VIN+
Routing:
- net 12V_REG: track 84.7 -> 107.2 mm
- net VIN_1: track 20.0 -> 15.8 mm
- net MAG_INC_N_1: track 11.0 -> 8.13 mm
- net N$3: track 15.6 -> 17.9 mm
- net N$29: track 10.1 -> 7.97 mm
- net VIN_2: track 19.7 -> 17.6 mm
- net PDIO_1: track 6.24 -> 8.21 mm
- net CSN_1: track 8.50 -> 6.75 mm
- net CSN_2: track 9.03 -> 7.34 mm
- net MAG_DEC_N_1: track 7.54 -> 6.02 mm
- net CLK_1: track 7.20 -> 5.73 mm
- net PDIO_2: track 6.90 -> 8.35 mm
- net N$4: track 9.38 -> 7.96 mm
- net CLK_2: track 8.17 -> 6.85 mm
- net MAG_DEC_N_2: track 8.49 -> 7.32 mm
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Other:
- board size 63.8 x 122 mm -> 63.5 x 122 mm
