File: task_12_PDS PCB/Power_Distro_Board_V4.sch (EAGLE design)
At the start: 62 parts

Commit message: Completed PDB Board
Parts:
- added C1_3: 100nF, resistor:C-EUC1206
- added C1_4: 10uF, resistor:C-EUC1206
- added ENC_2: ENCODER_AS5045B, minebot_PDR:ENCODER_AS5045B
- added MAIN_2, SUB_2: (no value), pinhead:PINHD-1X6
Connections:
- new net A_2: ENC_2.A, SUB_2.3
- new net B_2: ENC_2.B, SUB_2.4
- new net CLK_2: ENC_2.CLK, MAIN_2.4
- new net CSN_2: ENC_2.CSN, MAIN_2.3
- new net DO_2: ENC_2.DO, MAIN_2.5
- new net GND_2: C1_3.2, C1_4.2, ENC_2.VSS, MAIN_2.2
- new net I_2: ENC_2.I, SUB_2.5
- new net MAG_DEC_N_2: ENC_2.MAG_DEC_N, SUB_2.2
- new net MAG_INC_N_2: ENC_2.MAG_INC_N, SUB_2.1
- new net N$29: C1_4.1, ENC_2.VDD3V3
- new net PDIO_2: ENC_2.PDIO, SUB_2.6
- new net PWM_2: ENC_2.PWM, MAIN_2.6
- new net VIN_2: C1_3.1, ENC_2.VDD5V, MAIN_2.1
Other:
- note added: "**This encoder PCBs will be cut out of the main board"
- note removed: "**These 3 encoder PCBs will be cut out of the main board"
- note removed: "24V Output"

Commit message: PDB Final Updates
Parts:
- removed F1: 60VDC 50A, minebot_PDR:LITTLEFUSENANO463
- added F10: 20V, 50A, POWER_DISTRO:LITTLEFUSE_NANO
- F2, F3, F4, F5, F6, F7, F8, F9: device resistor:R-EU_R1206W -> resistor:R-EU_M1206
Connections:
- net 12V_REG: now also F10.OUT, TVS_1.C; no longer F1.VIN-, TVS_1.CATHODE
- net GND: now also TVS_1.A; no longer TVS_1.ANODE
- net N$3: now also F10.IN; no longer F1.VIN+
Changed lines of the file:
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@@
 <part name="GND10" library="supply1" library_urn="urn:adsk.eagle:library:371" deviceset="GND" device=""/>
 <part name="R10" library="resistor" library_urn="urn:adsk.eagle:library:348" deviceset="R-US_" device="R1206" package3d_urn="urn:adsk.eagle:package:26062/1" value="150"/>
-<part name="F1" library="minebot_PDR" deviceset="LITTLEFUSENANO463" device="" value="60VDC 50A"/>
 <part name="GND2" library="supply1" library_urn="urn:adsk.eagle:library:371" deviceset="GND" device=""/>
 <part name="GND14" library="supply1" library_urn="urn:adsk.eagle:library:371" deviceset="GND" device=""/>
@@
 <part name="PG2" library="testpad" library_urn="urn:adsk.eagle:library:385" deviceset="TP" device="PAD1-13" package3d_urn="urn:adsk.eagle:package:27946/1"/>
 <part name="EN2" library="testpad" library_urn="urn:adsk.eagle:library:385" deviceset="TP" device="PAD1-13" package3d_urn="urn:adsk.eagle:package:27946/1"/>
-<part name="F2" library="resistor" library_urn="urn:adsk.eagle:library:348" deviceset="R-EU_" device="R1206W" package3d_urn="urn:adsk.eagle:package:26064/1" value="60VDC 20A"/>
-<part name="F3" library="resistor" library_urn="urn:adsk.eagle:library:348" deviceset="R-EU_" device="R1206W" package3d_urn="urn:adsk.eagle:package:26064/1" value="60VDC 20A"/>
-<part name="F4" library="resistor" library_urn="urn:adsk.eagle:library:348" deviceset="R-EU_" device="R1206W" package3d_urn="urn:adsk.eagle:package:26064/1" value="60VDC 20A"/>
-<part name="F5" library="resistor" library_urn="urn:adsk.eagle:library:348" deviceset="R-EU_" device="R1206W" package3d_urn="urn:adsk.eagle:package:26064/1" value="60VDC 20A"/>
-<part name="F9" library="resistor" library_urn="urn:adsk.eagle:library:348" deviceset="R-EU_" device="R1206W" package3d_urn="urn:adsk.eagle:package:26064/1" value="60VDC 5A"/>
-<part name="F8" library="resistor" library_urn="urn:adsk.eagle:library:348" deviceset="R-EU_" device="R1206W" package3d_urn="urn:adsk.eagle:package:26064/1" value="60VDC 3A"/>
+<part name="F2" library="resistor" library_urn="urn:adsk.eagle:library:348" deviceset="R-EU_" device="M1206" package3d_urn="urn:adsk.eagle:package:26088/1" value="60VDC 20A"/>
+<part name="F3" library="resistor" library_urn="urn:adsk.eagle:library:348" deviceset="R-EU_" device="M1206" package3d_urn="urn:adsk.eagle:package:26088/1" value="60VDC 20A"/>
+<part name="F4" library="resistor" library_urn="urn:adsk.eagle:library:348" deviceset="R-EU_" device="M1206" package3d_urn="urn:adsk.eagle:package:26088/1" value="60VDC 20A"/>
+<part name="F5" library="resistor" library_urn="urn:adsk.eagle:library:348" deviceset="R-EU_" device="M1206" package3d_urn="urn:adsk.eagle:package:26088/1" value="60VDC 20A"/>
+<part name="F9" library="resistor" library_urn="urn:adsk.eagle:library:348" deviceset="R-EU_" device="M1206" package3d_urn="urn:adsk.eagle:package:26088/1" value="60VDC 5A"/>
+<part name="F8" library="resistor" library_urn="urn:adsk.eagle:library:348" deviceset="R-EU_" device="M1206" package3d_urn="urn:adsk.eagle:package:26088/1" value="60VDC 3A"/>
 <part name="MOTOR_OUT_5" library="con-molex" library_urn="urn:adsk.eagle:library:165" deviceset="5566-2" device=""/>
 <part name="12V_5" library="led" library_urn="urn:adsk.eagle:library:259" deviceset="LED" device="SML1206" package3d_urn="urn:adsk.eagle:package:15829/1" value="GREEN"/>
@@
 <part name="GND5" library="supply1" library_urn="urn:adsk.eagle:library:371" deviceset="GND" device=""/>
 <part name="GND11" library="supply1" library_urn="urn:adsk.eagle:library:371" deviceset="GND" device=""/>
-<part name="F6" library="resistor" library_urn="urn:adsk.eagle:library:348" deviceset="R-EU_" device="R1206W" package3d_urn="urn:adsk.eagle:package:26064/1" value="60VDC 20A"/>
+<part name="F6" library="resistor" library_urn="urn:adsk.eagle:library:348" deviceset="R-EU_" device="M1206" package3d_urn="urn:adsk.eagle:package:26088/1" value="60VDC 20A"/>
 <part name="MOTOR_OUT_6" library="con-molex" library_urn="urn:adsk.eagle:library:165" deviceset="5566-2" device=""/>
 <part name="12V_6" library="led" library_urn="urn:adsk.eagle:library:259" deviceset="LED" device="SML1206" package3d_urn="urn:adsk.eagle:package:15829/1" value="GREEN"/>
@@
 <part name="GND12" library="supply1" library_urn="urn:adsk.eagle:library:371" deviceset="GND" device=""/>
 <part name="GND13" library="supply1" library_urn="urn:adsk.eagle:library:371" deviceset="GND" device=""/>
-<part name="F7" library="resistor" library_urn="urn:adsk.eagle:library:348" deviceset="R-EU_" device="R1206W" package3d_urn="urn:adsk.eagle:package:26064/1" value="60VDC 20A"/>
+<part name="F7" library="resistor" library_urn="urn:adsk.eagle:library:348" deviceset="R-EU_" device="M1206" package3d_urn="urn:adsk.eagle:package:26088/1" value="60VDC 20A"/>
 <part name="ENC_2" library="minebot_PDR" deviceset="ENCODER_AS5045B" device=""/>
 <part name="C1_3" library="resistor" library_urn="urn:adsk.eagle:library:348" deviceset="C-EU" device="C1206" package3d_urn="urn:adsk.eagle:package:26140/1" value="100nF"/>
@@
 <part name="MAIN_2" library="pinhead" library_urn="urn:adsk.eagle:library:325" deviceset="PINHD-1X6" device="" package3d_urn="urn:adsk.eagle:package:22472/2"/>
 <part name="SUB_2" library="pinhead" library_urn="urn:adsk.eagle:library:325" deviceset="PINHD-1X6" device="" package3d_urn="urn:adsk.eagle:package:22472/2"/>
+<part name="F10" library="POWER_DISTRO" deviceset="LITTLEFUSE_NANO" device="" value="20V, 50A"/>
 </parts>
 <sheets>
@@
 <attribute name="VALUE" x="105.41" y="-39.878" size="1.778" layer="96" rot="R180"/>
 </instance>
-<instance part="F1" gate="G$1" x="30.48" y="55.88"/>
 <instance part="GND2" gate="1" x="53.34" y="-55.88"/>
 <instance part="GND14" gate="1" x="55.88" y="-7.62"/>
@@
 <instance part="MAIN_2" gate="A" x="297.18" y="5.08"/>
 <instance part="SUB_2" gate="A" x="350.52" y="5.08"/>
+<instance part="F10" gate="G$1" x="30.48" y="55.88"/>
 </instances>
 <busses>
@@
 <segment>
 <pinref part="PWR_IN" gate="-2" pin="S"/>
-<pinref part="TVS_1" gate="G$1" pin="ANODE"/>
+<pinref part="TVS_1" gate="G$1" pin="A"/>
 <wire x1="12.7" y1="76.2" x2="71.12" y2="76.2" width="0.1524" layer="91"/>
 <pinref part="GND3" gate="1" pin="GND"/>
@@
 <pinref part="PWR_IN" gate="-1" pin="S"/>
 <wire x1="10.16" y1="55.88" x2="15.24" y2="55.88" width="0.1524" layer="91"/>
-<pinref part="F1" gate="G$1" pin="VIN+"/>
 <wire x1="15.24" y1="55.88" x2="17.78" y2="55.88" width="0.1524" layer="91"/>
 <junction x="15.24" y="55.88"/>
+<pinref part="F10" gate="G$1" pin="IN"/>
 </segment>
 </net>
@@
 <net name="12V_REG" class="0">
 <segment>
-<pinref part="TVS_1" gate="G$1" pin="CATHODE"/>
+<pinref part="TVS_1" gate="G$1" pin="C"/>
 <label x="71.12" y="48.26" size="1.778" layer="95"/>
 <junction x="71.12" y="55.88"/>
@@
 <wire x1="106.68" y1="55.88" x2="106.68" y2="63.5" width="0.1524" layer="91"/>
 <wire x1="88.9" y1="55.88" x2="106.68" y2="55.88" width="0.1524" layer="91"/>
-<pinref part="F1" gate="G$1" pin="VIN-"/>
 <wire x1="43.18" y1="55.88" x2="45.72" y2="55.88" width="0.1524" layer="91"/>
 <junction x="45.72" y="55.88"/>
@@
 <junction x="157.48" y="73.66"/>
 <junction x="157.48" y="48.26"/>
-</segment>
-</net>
+<pinref part="F10" gate="G$1" pin="OUT"/>
+</segment>
+</net>
